Commit message: fix: 修正urdf和xml质量参数

File: src/wheel_legged_description/zt_2025_Infantry_wheelLegged/urdf/zt_2025_Infantry_wheelLeggedP_withShoot_s.urdf (robot description, URDF)
Before this commit: robot RMInfantry_Complation_Vision.SLDASM, 20 links, 19 joints
Links:
- link base_link: mass 9.774 -> 16.77493621
- link left_chassis_wheel_link: mass 0.52417 -> 1.24506308
- link left_front_hip_link: mass 0.2528 -> 0.25279841
- link left_front_knee_link: mass 0.21937 -> 0.21937234
- link left_rear_hip_link: mass 0.258169857475487 -> 0.25816986
- link left_rear_knee_link: mass 0.2214 -> 0.22140128
- link right_front_hip_link: mass 0.2528 -> 0.25279841
- link right_front_knee_link: mass 0.21937 -> 0.21937234
- link right_rear_hip_link: mass 0.25817 -> 0.25816986
- link right_rear_knee_link: mass 0.2214 -> 0.22140128

Commit message: fix: 修正质量参数并重新整定相关参数
-修复urdf和xml文件关于sw导出质量参数问题
-按照1新的质量参数重新整定LQR参数

File: src/wheel_legged_description/zt_2025_Infantry_wheelLegged/urdf/zt_2025_Infantry_wheelLeggedP_withShoot_s.urdf (robot description, URDF)
Before this commit: robot RMInfantry_Complation_Vision.SLDASM, 20 links, 19 joints
Links:
- link gimbal_pitch_link: mass 1.26308074496479 -> 2.23648116
- link gimbal_pitch_motor_link: mass 0.29161 -> 0.48928842
- link gimbal_yaw_link: mass 0.70223 -> 0.70223299
- link right_chassis_wheel_link: mass 0.52417 -> 1.24506308
