Commit message: chore: 修改为ROS2 pkg

File: src/wheel_legged_description/Infantry_wheelLegged_cyclBot/urdf/zt_2025_Infantry_wheelLeggedP_withShoot_s.urdf (robot description, URDF)
Before this commit: robot RMInfantry_Complation_Vision.SLDASM, 20 links, 19 joints
Joints:
- removed joint floating_base_joint
- added joint world_to_base: type fixed, parent world, child base_link, origin xyz=0 0 0 rpy=0 0 0
